File: kicad/rainguage-v2/rainguage.kicad_pcb (KiCad board)
At the start: 2 copper layers, 31.3 x 61.4 mm, 22 parts, among them J1 Hall sensor Connector, J2 Connecteur USB (+5v), J3 Con. LiPO battery, Q1 2N7002, U1 MCP73831-2-OT, U2 ATtiny85-20P, U3 DRV5033FAxDBZ, U4 CR2450

Commit message: Update doc
Parts:
- removed U3: DRV5033FAxDBZ, Package_TO_SOT_SMD:SOT-23
- removed U4: CR2450, Battery:BatteryHolder_ComfortableElectronic_CH273-2450_1x2450
- added H1: MountingHole_Pad, MountingHole:MountingHole_2.2mm_M2_Pad, F.Cu at (159.6, 62.9)
- added H2: MountingHole_Pad, MountingHole:MountingHole_2.2mm_M2_Pad, F.Cu at (186.9, 62.9)
- added H3: MountingHole_Pad, MountingHole:MountingHole_2.2mm_M2_Pad, F.Cu at (159.6, 118.2)
- added H4: MountingHole_Pad, MountingHole:MountingHole_2.2mm_M2_Pad, F.Cu at (186.9, 118.5)
- added J4: Hall sensor Connector 3, Connector_PinSocket_2.54mm:PinSocket_1x03_P2.54mm_Vertical, F.Cu at (170.6, 75.4)
- added J5: Hall sensor Connector 2, Connector_PinSocket_2.54mm:PinSocket_1x03_P2.54mm_Vertical, F.Cu at (170.6, 71.7)
- added J6: Hall sensor Connector 4, Connector_PinSocket_2.54mm:PinSocket_1x03_P2.54mm_Vertical, F.Cu at (170.6, 68.0)
- J1: value Hall sensor Connector -> Hall sensor Connector 1
- J2: value Connecteur USB (+5v) -> Con. USB (+5v)
- R1: value 2kOhm -> 2k Ohm
- R2: value 470Ohm -> 470 Ohm
- moved C5 28.7 mm to (187.1, 113.4)
- moved L2 16.5 mm to (182.5, 107.2), turned to 0 degrees
- moved C3 13.6 mm to (181.4, 110.9), turned to 0 degrees
- moved R1 10.8 mm to (166.0, 110.7), turned to 180 degrees
- moved C2 6.98 mm to (159.1, 113.6)
- moved D1 5.40 mm to (161.4, 113.6)
- moved D2 4.81 mm to (187.1, 105.7), turned to 90 degrees
- moved R2 3.42 mm to (159.1, 109.2), turned to -90 degrees
- moved J2 2.97 mm to (165.0, 117.4)
- moved U1 2.66 mm to (164.9, 107.8), turned to 180 degrees
- moved R6 2.57 mm to (178.6, 97.2), turned to 180 degrees
- moved C1 2.50 mm to (166.0, 104.1), turned to 90 degrees
- moved J1 1.44 mm to (171.1, 117.7)
- moved Q1 1.35 mm to (178.6, 100.3), turned to -90 degrees
- moved R5 1.30 mm to (173.0, 104.0)
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Routing:
- net VBAT: track 0.00 -> 75.9 mm, vias 0 -> 1
- net +3.3v: track 4.27 -> 74.0 mm
- net PB2: track 0.00 -> 52.2 mm, vias 0 -> 1
- net PB1: track 0.00 -> 30.5 mm
- net PB0: track 0.00 -> 19.0 mm
- net USB 5V: track 0.00 -> 17.9 mm
- net GND: track 0.00 -> 17.7 mm
- net Net-(U1-STAT): track 0.00 -> 14.6 mm, vias 0 -> 2
- net Net-(D2-A): track 0.00 -> 14.0 mm
- net Net-(U2-XTAL1/PB3): track 0.00 -> 5.16 mm
- net Net-(D1-K): track 0.00 -> 4.07 mm
- net Net-(Q1-D): track 0.00 -> 3.10 mm
- net Net-(U1-PROG): track 0.00 -> 2.61 mm
- net Net-(D2-K): track 0.00 -> 2.01 mm
- added copper zone on B.Cu, net GND
- added copper zone on F.Cu, net GND
Other:
- board size 31.3 x 61.4 mm -> 33.1 x 61.4 mm
- board text added: "+3.3v"
- board text added: "GND"
- board text added: "Hall effect sensor"
- board text added: "JLCJLCJLCJLC"
- board text added: "Raingauge Mark II Guiet - 12/2023"
- board text added: "Sensor"
- board text added: "USB (+5v)"
- board text added: "Vbat"
- board text added: "XBEE"

Commit message: update doc
Connections:
- J4 pad 2: PB2 -> GND
- J4 pad 3: GND -> PB2
- J5 pad 2: PB2 -> GND
- J5 pad 3: GND -> PB2
- J6 pad 2: PB2 -> GND
- J6 pad 3: GND -> PB2
Routing:
- net PB2: track 52.2 -> 51.6 mm
Changed lines of the file:
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@@
       (net 4 "+3.3v") (pinfunction "Pin_1") (pintype "passive"))
     (pad "2" thru_hole oval (at 0 2.54 90) (size 1.7 1.7) (drill 1) (layers "*.Cu" "*.Mask")
-      (net 16 "PB2") (pinfunction "Pin_2") (pintype "passive"))
+      (net 2 "GND") (pinfunction "Pin_2") (pintype "passive"))
     (pad "3" thru_hole oval (at 0 5.08 90) (size 1.7 1.7) (drill 1) (layers "*.Cu" "*.Mask")
-      (net 2 "GND") (pinfunction "Pin_3") (pintype "passive"))
+      (net 16 "PB2") (pinfunction "Pin_3") (pintype "passive"))
     (model "${KICAD6_3DMODEL_DIR}/Connector_PinSocket_2.54mm.3dshapes/PinSocket_1x03_P2.54mm_Vertical.wrl"
       (offset (xyz 0 0 0))
@@
       (net 4 "+3.3v") (pinfunction "Pin_1") (pintype "passive"))
     (pad "2" thru_hole oval (at 0 2.54 90) (size 1.7 1.7) (drill 1) (layers "*.Cu" "*.Mask")
-      (net 16 "PB2") (pinfunction "Pin_2") (pintype "passive"))
+      (net 2 "GND") (pinfunction "Pin_2") (pintype "passive"))
     (pad "3" thru_hole oval (at 0 5.08 90) (size 1.7 1.7) (drill 1) (layers "*.Cu" "*.Mask")
-      (net 2 "GND") (pinfunction "Pin_3") (pintype "passive"))
+      (net 16 "PB2") (pinfunction "Pin_3") (pintype "passive"))
     (model "${KICAD6_3DMODEL_DIR}/Connector_PinSocket_2.54mm.3dshapes/PinSocket_1x03_P2.54mm_Vertical.wrl"
       (offset (xyz 0 0 0))
@@
       (net 4 "+3.3v") (pinfunction "Pin_1") (pintype "passive"))
     (pad "2" thru_hole oval (at 0 2.54 90) (size 1.7 1.7) (drill 1) (layers "*.Cu" "*.Mask")
-      (net 16 "PB2") (pinfunction "Pin_2") (pintype "passive"))
+      (net 2 "GND") (pinfunction "Pin_2") (pintype "passive"))
     (pad "3" thru_hole oval (at 0 5.08 90) (size 1.7 1.7) (drill 1) (layers "*.Cu" "*.Mask")
-      (net 2 "GND") (pinfunction "Pin_3") (pintype "passive"))
+      (net 16 "PB2") (pinfunction "Pin_3") (pintype "passive"))
     (model "${KICAD6_3DMODEL_DIR}/Connector_PinSocket_2.54mm.3dshapes/PinSocket_1x03_P2.54mm_Vertical.wrl"
       (offset (xyz 0 0 0))
@@
   (segment (start 173.228 88.9) (end 176.911 88.9) (width 0.8) (layer "B.Cu") (net 1))
   (segment (start 157.578276 105.311724) (end 157.578276 111.101276) (width 0.8) (layer "F.Cu") (net 2))
+  (segment (start 173.101 75.555) (end 173.116 75.54) (width 0.4) (layer "F.Cu") (net 2))
   (segment (start 159.89554 102.99446) (end 157.578276 105.311724) (width 0.8) (layer "F.Cu") (net 2))
   (segment (start 157.578276 111.101276) (end 159.131 112.654) (width 0.8) (layer "F.Cu") (net 2))
@@
   (segment (start 173.466 105.902) (end 171.069 103.505) (width 0.4) (layer "B.Cu") (net 15))
   (segment (start 171.069 98.03638) (end 162.0266 88.99398) (width 0.4) (layer "B.Cu") (net 15))
-  (segment (start 173.116 75.413) (end 173.116 71.73) (width 0.4) (layer "F.Cu") (net 16))
   (segment (start 175.006 99.06) (end 175.006 80.264) (width 0.4) (layer "F.Cu") (net 16))
-  (segment (start 173.101 78.359) (end 173.116 78.344) (width 0.4) (layer "F.Cu") (net 16))
-  (segment (start 175.006 80.264) (end 173.101 78.359) (width 0.4) (layer "F.Cu") (net 16))
-  (segment (start 173.101 75.555) (end 173.116 75.54) (width 0.4) (layer "F.Cu") (net 16))
+  (segment (start 175.656 71.73) (end 175.656 68.047) (width 0.4) (layer "F.Cu") (net 16))
+  (segment (start 175.656 79.614) (end 175.656 75.413) (width 0.4) (layer "F.Cu") (net 16))
   (segment (start 174.879 116.468003) (end 173.609 117.738003) (width 0.4) (layer "F.Cu") (net 16))
-  (segment (start 173.116 78.344) (end 173.116 75.413) (width 0.4) (layer "F.Cu") (net 16))
   (segment (start 174.879 114.3) (end 174.879 116.468003) (width 0.4) (layer "F.Cu") (net 16))
-  (segment (start 173.116 71.73) (end 173.116 68.047) (width 0.4) (layer "F.Cu") (net 16))
+  (segment (start 175.656 75.413) (end 175.656 71.73) (width 0.4) (layer "F.Cu") (net 16))
+  (segment (start 175.006 80.264) (end 175.656 79.614) (width 0.4) (layer "F.Cu") (net 16))
   (via (at 175.006 99.06) (size 0.6) (drill 0.3) (layers "F.Cu" "B.Cu") (net 16))
   (segment (start 174.879 114.3) (end 176.292 112.887) (width 0.4) (layer "B.Cu") (net 16))
