File: kicad/rainguage-v2/rainguage.kicad_sch (KiCad schematic)
At the start: 13 parts, among them J2 Connecteur USB (+5v), J3 Con. LiPO battery, U1 MCP73831-2-OT, U2 ATtiny85-20P

Commit message: commit des familles
Parts:
- added D2: LED, LED_SMD:LED_0805_2012Metric, symbol Device:LED
- added H1, H2, H3, H4: MountingHole_Pad, MountingHole:MountingHole_2.2mm_M2_Pad_Via, symbol Mechanical:MountingHole_Pad
- added J1: Hall sensor Connector, Connector_JST:JST_EH_B3B-EH-A_1x03_P2.50mm_Vertical, symbol Connector_Generic:Conn_01x03
- added Q1: 2N7002, Package_TO_SOT_SMD:SOT-23, symbol Transistor_FET:2N7002
- added R3: 100Ohm, Resistor_SMD:R_0805_2012Metric, symbol Device:R
- added R4: 3.3kOhm, Resistor_SMD:R_0805_2012Metric, symbol Device:R
- added R5, R6: 10kOhm, Resistor_SMD:R_0805_2012Metric, symbol Device:R
- added U3: DRV5033FAxDBZ, Package_TO_SOT_SMD:SOT-23, symbol Sensor_Magnetic:DRV5033FAxDBZ
- added U4: CR2450, Battery:BatteryHolder_ComfortableElectronic_CH273-2450_1x2450, symbol raingauge-v2-3:CR2450
- C1, C2, C3, C5: footprint (none) -> Capacitor_SMD:C_0805_2012Metric
- D1: footprint (none) -> LED_SMD:LED_0805_2012Metric
- J2, J3: footprint (none) -> Connector_JST:JST_EH_B2B-EH-A_1x02_P2.50mm_Vertical
- JP1: footprint XBEE -> RF:XBEE
- L2: footprint (none) -> Package_TO_SOT_SMD:SOT-89-3
- R1, R2: footprint (none) -> Resistor_SMD:R_0805_2012Metric
Connections:
- net +3.3v: now also C3.1, JP1.1 (VDD), L2.3 (VOUT), U2.8 (VCC), J1.3 (Pin_3), U3.1 (VCC); no longer C5.1, L2.2 (VIN)
- net GND: now also JP1.10 (GND), U2.4 (GND), J1.1 (Pin_1), Q1.2 (S), R3.2, R6.2, U3.3 (GND), U4.2 (-)
- net VBAT: now also C5.1, L2.2 (VIN), R5.2, U4.1 (+); no longer C3.1, L2.3 (VOUT)
- net at U2.2 (XTAL1/PB3): now also R4.2, R5.1
- net PB0: now reaches U2.5 (AREF/PB0)
- net PB0: now also JP1.9 (DTR)
- net PB1: now reaches U2.6 (PB1)
- net PB1: now also JP1.3 (DIN)
- net PB2: now reaches U2.7 (PB2)
- net PB2: now also J1.2 (Pin_2), U3.2 (OUT)
- net at JP1.13 (DIO9): now also D2.2 (A), Q1.1 (G), R6.1
- new net: D2.1 (K), R3.1
- new net: Q1.3 (D), R4.1
- no-connect marks 0 -> 17
Other:
- note added: "ATtiny 85"
- note added: "Alimentation"
- note added: "Hall Sensor"
- note added: "Mounting holes"
- note added: "XBEE"
- moved on the sheet: JP1

Commit message: Update doc
Parts:
- removed U4: CR2450, Battery:BatteryHolder_ComfortableElectronic_CH273-2450_1x2450, symbol raingauge-v2-3:CR2450
- added J4: Hall sensor Connector 3, Connector_PinSocket_2.54mm:PinSocket_1x03_P2.54mm_Vertical, symbol Connector:Conn_01x03_Pin
- added J5: Hall sensor Connector 2, Connector_PinSocket_2.54mm:PinSocket_1x03_P2.54mm_Vertical, symbol Connector:Conn_01x03_Pin
- added J6: Hall sensor Connector 4, Connector_PinSocket_2.54mm:PinSocket_1x03_P2.54mm_Vertical, symbol Connector:Conn_01x03_Pin
- H1, H2, H3, H4: footprint MountingHole:MountingHole_2.2mm_M2_Pad_Via -> MountingHole:MountingHole_2.2mm_M2_Pad
- J1: value Hall sensor Connector -> Hall sensor Connector 1
- J2: value Connecteur USB (+5v) -> Con. USB (+5v)
- R1: value 2kOhm -> 2k Ohm
- R2: value 470Ohm -> 470 Ohm
Connections:
- net +3.3v: now also J4.1 (Pin_1), J5.1 (Pin_1), J6.1 (Pin_1)
- net GND: now also H1.1, H2.1, H3.1, H4.1, J4.3 (Pin_3), J5.3 (Pin_3), J6.3 (Pin_3)
- net PB2: now also J4.2 (Pin_2), J5.2 (Pin_2), J6.2 (Pin_2)
Other:
- moved on the sheet: H3, H4, J1, U3

Commit message: update doc
Connections:
- net GND: now also J4.2 (Pin_2), J5.2 (Pin_2), J6.2 (Pin_2); no longer J4.3 (Pin_3), J5.3 (Pin_3), J6.3 (Pin_3)
- net PB2: now also J4.3 (Pin_3), J5.3 (Pin_3), J6.3 (Pin_3); no longer J4.2 (Pin_2), J5.2 (Pin_2), J6.2 (Pin_2)
Changed lines of the file:
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@@
+    )
+  )
+  (global_label "PB2" (shape input) (at 207.01 142.24 90) (fields_autoplaced)
+    (effects (font (size 1.27 1.27)) (justify left))
+    (property "Intersheetrefs" "${INTERSHEET_REFS}" (at 207.01 135.5053 90)
+      (effects (font (size 1.27 1.27)) (justify left) hide)
     )
   )
@@
     )
   )
-  (global_label "PB2" (shape input) (at 232.41 146.05 90) (fields_autoplaced)
-    (effects (font (size 1.27 1.27)) (justify left))
-    (property "Intersheetrefs" "${INTERSHEET_REFS}" (at 232.41 139.3153 90)
-      (effects (font (size 1.27 1.27)) (justify left) hide)
-    )
-  )
   (global_label "+3.3v" (shape input) (at 199.39 146.05 90) (fields_autoplaced)
     (effects (font (size 1.27 1.27)) (justify left))
     (property "Intersheetrefs" "${INTERSHEET_REFS}" (at 199.39 137.501 90)
-      (effects (font (size 1.27 1.27)) (justify left) hide)
-    )
-  )
-  (global_label "PB2" (shape input) (at 256.54 123.19 90) (fields_autoplaced)
-    (effects (font (size 1.27 1.27)) (justify left))
-    (property "Intersheetrefs" "${INTERSHEET_REFS}" (at 256.54 116.4553 90)
-      (effects (font (size 1.27 1.27)) (justify left) hide)
-    )
-  )
-  (global_label "PB2" (shape input) (at 203.2 146.05 90) (fields_autoplaced)
-    (effects (font (size 1.27 1.27)) (justify left))
-    (property "Intersheetrefs" "${INTERSHEET_REFS}" (at 203.2 139.3153 90)
       (effects (font (size 1.27 1.27)) (justify left) hide)
     )
@@
     (effects (font (size 1.27 1.27)) (justify left))
     (property "Intersheetrefs" "${INTERSHEET_REFS}" (at 214.63 90.511 90)
+      (effects (font (size 1.27 1.27)) (justify left) hide)
+    )
+  )
+  (global_label "PB2" (shape input) (at 260.35 119.38 90) (fields_autoplaced)
+    (effects (font (size 1.27 1.27)) (justify left))
+    (property "Intersheetrefs" "${INTERSHEET_REFS}" (at 260.35 112.6453 90)
+      (effects (font (size 1.27 1.27)) (justify left) hide)
+    )
+  )
+  (global_label "PB2" (shape input) (at 236.22 142.24 90) (fields_autoplaced)
+    (effects (font (size 1.27 1.27)) (justify left))
+    (property "Intersheetrefs" "${INTERSHEET_REFS}" (at 236.22 135.5053 90)
       (effects (font (size 1.27 1.27)) (justify left) hide)
     )
@@
         (path "/cf99271c-479e-4771-be01-83565bacf100"
           (reference "#PWR04") (unit 1)
-        )
-      )
-    )
-  )
-  (symbol (lib_id "power:GND") (at 236.22 142.24 180) (unit 1)
-    (in_bom yes) (on_board yes) (dnp no) (fields_autoplaced)
-    (property "Reference" "#PWR012" (at 236.22 135.89 0)
-      (effects (font (size 1.27 1.27)) hide)
-    )
-    (property "Value" "GND" (at 236.22 137.16 0)
-      (effects (font (size 1.27 1.27)))
-    )
-    (property "Footprint" "" (at 236.22 142.24 0)
-      (effects (font (size 1.27 1.27)) hide)
-    )
-    (property "Datasheet" "" (at 236.22 142.24 0)
-      (effects (font (size 1.27 1.27)) hide)
-    )
-    (pin "1")
-    (instances
-      (project "rainguage"
-        (path "/cf99271c-479e-4771-be01-83565bacf100"
-          (reference "#PWR012") (unit 1)
-        )
-      )
-    )
-  )
-  (symbol (lib_id "power:GND") (at 207.01 142.24 180) (unit 1)
-    (in_bom yes) (on_board yes) (dnp no) (fields_autoplaced)
-    (property "Reference" "#PWR019" (at 207.01 135.89 0)
-      (effects (font (size 1.27 1.27)) hide)
-    )
-    (property "Value" "GND" (at 207.01 137.16 0)
-      (effects (font (size 1.27 1.27)))
-    )
-    (property "Footprint" "" (at 207.01 142.24 0)
-      (effects (font (size 1.27 1.27)) hide)
-    )
-    (property "Datasheet" "" (at 207.01 142.24 0)
-      (effects (font (size 1.27 1.27)) hide)
-    )
-    (pin "1")
-    (instances
-      (project "rainguage"
-        (path "/cf99271c-479e-4771-be01-83565bacf100"
-          (reference "#PWR019") (unit 1)
         )
       )
@@
     )
   )
+  (symbol (lib_id "power:GND") (at 232.41 146.05 180) (unit 1)
+    (in_bom yes) (on_board yes) (dnp no) (fields_autoplaced)
+    (property "Reference" "#PWR012" (at 232.41 139.7 0)
+      (effects (font (size 1.27 1.27)) hide)
+    )
+    (property "Value" "GND" (at 232.41 140.97 0)
+      (effects (font (size 1.27 1.27)))
+    )
+    (property "Footprint" "" (at 232.41 146.05 0)
+      (effects (font (size 1.27 1.27)) hide)
+    )
+    (property "Datasheet" "" (at 232.41 146.05 0)
+      (effects (font (size 1.27 1.27)) hide)
+    )
+    (pin "1")
+    (instances
+      (project "rainguage"
+        (path "/cf99271c-479e-4771-be01-83565bacf100"
+          (reference "#PWR012") (unit 1)
+        )
+      )
+    )
+  )
+  (symbol (lib_id "power:GND") (at 256.54 123.19 180) (unit 1)
+    (in_bom yes) (on_board yes) (dnp no) (fields_autoplaced)
+    (property "Reference" "#PWR020" (at 256.54 116.84 0)
+      (effects (font (size 1.27 1.27)) hide)
+    )
+    (property "Value" "GND" (at 256.54 118.11 0)
+      (effects (font (size 1.27 1.27)))
+    )
+    (property "Footprint" "" (at 256.54 123.19 0)
+      (effects (font (size 1.27 1.27)) hide)
+    )
+    (property "Datasheet" "" (at 256.54 123.19 0)
+      (effects (font (size 1.27 1.27)) hide)
+    )
+    (pin "1")
+    (instances
+      (project "rainguage"
+        (path "/cf99271c-479e-4771-be01-83565bacf100"
+          (reference "#PWR020") (unit 1)
+        )
+      )
+    )
+  )
   (symbol (lib_id "power:GND") (at 254 41.91 0) (unit 1)
     (in_bom yes) (on_board yes) (dnp no)
@@
     )
   )
-  (symbol (lib_id "power:GND") (at 260.35 119.38 180) (unit 1)
-    (in_bom yes) (on_board yes) (dnp no) (fields_autoplaced)
-    (property "Reference" "#PWR020" (at 260.35 113.03 0)
-      (effects (font (size 1.27 1.27)) hide)
-    )
-    (property "Value" "GND" (at 260.35 114.3 0)
-      (effects (font (size 1.27 1.27)))
-    )
-    (property "Footprint" "" (at 260.35 119.38 0)
-      (effects (font (size 1.27 1.27)) hide)
-    )
-    (property "Datasheet" "" (at 260.35 119.38 0)
-      (effects (font (size 1.27 1.27)) hide)
-    )
-    (pin "1")
-    (instances
-      (project "rainguage"
-        (path "/cf99271c-479e-4771-be01-83565bacf100"
-          (reference "#PWR020") (unit 1)
-        )
-      )
-    )
-  )
   (symbol (lib_id "power:GND") (at 71.12 29.21 180) (unit 1)
     (in_bom yes) (on_board yes) (dnp no) (fields_autoplaced)
@@
         )
       )
+    )
+  )
+  (symbol (lib_id "power:GND") (at 203.2 146.05 180) (unit 1)
+    (in_bom yes) (on_board yes) (dnp no) (fields_autoplaced)
+    (property "Reference" "#PWR019" (at 203.2 139.7 0)
+      (effects (font (size 1.27 1.27)) hide)
+    )
+    (property "Value" "GND" (at 203.2 140.97 0)
+      (effects (font (size 1.27 1.27)))
+    )
+    (property "Footprint" "" (at 203.2 146.05 0)
+      (effects (font (size 1.27 1.27)) hide)
+    )
+    (property "Datasheet" "" (at 203.2 146.05 0)
+      (effects (font (size 1.27 1.27)) hide)
+    )
+    (pin "1")
+    (instances
+      (project "rainguage"
+        (path "/cf99271c-479e-4771-be01-83565bacf100"
+          (reference "#PWR019") (unit 1)
+        )
+      )

Commit message: Update doc
Parts:
- R3: value 100Ohm -> 100 Ohm
Changed lines of the file:
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@@
       (effects (font (size 1.27 1.27)))
     )
-    (property "Value" "100Ohm" (at 182.88 115.57 90)
+    (property "Value" "100 Ohm" (at 182.88 115.57 90)
       (effects (font (size 1.27 1.27)))
     )
